File: 68k_20_to_30.kicad_sch (KiCad schematic)
At the start: 3 parts, among them U1 68030

Commit message: Adding current state of routing.
Parts:
- added R2, R3, R4: R1k, Resistor_THT:R_Axial_DIN0204_L3.6mm_D1.6mm_P5.08mm_Horizontal, symbol Device:R
- U2: value ~ -> 68020
Connections:
- net VCC: now also R2.1, R3.2, R4.2
- new net: R1.2, U1.L1 (CIIN)
- new net: R4.1, U1.F13 (MMUDIS)
- new net: R3.1, U1.G1 (STERM)
- new net: R2.2, U1.J1 (CBACK)
Other:
- moved on the sheet: R1
