File: 68k_20_to_30_hand_route.kicad_pcb (KiCad board)
At the start: 4 copper layers, 86 x 78.5 mm, 6 parts, among them U1 68030, U2 68020

Commit message: Adding current state of routing.
Routing:
- net /D3: track 0.00 -> 68.4 mm
- net /D8: track 0.00 -> 64.2 mm
- net /D2: track 0.00 -> 61.3 mm
- net /D0: track 0.00 -> 59.0 mm
- net /IPL0: track 0.00 -> 57.8 mm
- net /A15: track 0.00 -> 52.0 mm
- net /A8: track 0.00 -> 51.5 mm
- net /IPL1: track 0.00 -> 51.3 mm
- net /A10: track 0.00 -> 47.7 mm
- net /IPEND: track 0.00 -> 44.0 mm
- net /A2: track 0.00 -> 43.1 mm
- net /D22: track 0.00 -> 42.9 mm
- net /A3: track 0.00 -> 42.4 mm
- net /D19: track 0.00 -> 41.6 mm
- net /D20: track 0.00 -> 41.5 mm
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Other:
- board size 86 x 78.5 mm -> 123.6 x 78.5 mm
