File: 68k_20_to_30_no_vcc_plane.kicad_pcb (KiCad board)
At the start: 4 copper layers, 86 x 78.5 mm, 6 parts, among them U1 68030, U2 68020

Commit message: Adding current state of routing.
Routing:
- removed copper zone on In1.Cu, net VCC
Changed lines of the file:
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@@
 		(tags "Resistor Axial_DIN0204 series Axial Horizontal pin pitch 5.08mm 0.167W length 3.6mm diameter 1.6mm")
 		(property "Reference" "R3"
-			(at 2.54 1.85 360)
+			(at 2.54 1.85 0)
 			(layer "F.SilkS")
 			(effects
@@
 		)
 		(property "Value" "R1k"
-			(at 2.54 1.92 360)
+			(at 2.54 1.92 0)
 			(layer "F.Fab")
 			(effects
@@
 		)
 		(fp_text user "${REFERENCE}"
-			(at 2.54 0 360)
+			(at 2.54 0 0)
 			(layer "F.Fab")
 			(effects
@@
 	)
 	(zone
-		(net 1)
-		(net_name "VCC")
-		(layer "In1.Cu")
-		(name "VCC")
-		(hatch edge 0.5)
-		(connect_pads
-			(clearance 0.25)
-		)
-		(min_thickness 0.25)
-		(filled_areas_thickness no)
-		(fill yes
-			(thermal_gap 0.5)
-			(thermal_bridge_width 0.5)
-		)
-		(polygon
-			(pts
-				(xy 110 51) (xy 166 51) (xy 166 129.4) (xy 110 129.4)
-			)
-		)
-	)
-	(zone
